Commit message: commit changes to joint

File: body.urdf (robot description, URDF)
Before this commit: robot robot, 2 links, 0 joints
Links:
- removed link Leg
- added link BackLeg, mass 1; collision box size=1 1 1; visual box size=1 1 1
- added link FrontLeg, mass 1; collision box size=1 1 1; visual box size=1 1 1
Joints:
- added joint BackLeg_Torso: type revolute, parent BackLeg, child Torso, origin xyz=0.0 0.5 1.0 rpy=0 0 0, axis 0 1 0, limit lower=-3.14159 upper=3.14159 effort=0.0 velocity=0.0
- added joint Torso_FrontLeg: type revolute, parent Torso, child FrontLeg, origin xyz=0.0 0.5 -0.5 rpy=0 0 0, axis 0 1 0, limit lower=-3.14159 upper=3.14159 effort=0.0 velocity=0.0

Commit message: commit

File: body.urdf (robot description, URDF)
Before this commit: robot robot, 3 links, 2 joints
Joints:
- joint BackLeg_Torso: origin xyz=0.0 0.5 1.0 rpy=0 0 0 -> xyz=1.0 0 1.0 rpy=0 0 0

Commit message: changes + analyse.py

File: body.urdf (robot description, URDF)
Before this commit: robot robot, 3 links, 2 joints
Joints:
- removed joint BackLeg_Torso
- added joint Torso_BackLeg: type revolute, parent Torso, child BackLeg, origin xyz=1.0 0 1.0 rpy=0 0 0, axis 0 1 0, limit lower=-3.14159 upper=3.14159 effort=0.0 velocity=0.0
- joint Torso_FrontLeg: origin xyz=0.0 0.5 -0.5 rpy=0 0 0 -> xyz=2 0 1 rpy=0 0 0

Commit message: commit

File: body.urdf (robot description, URDF)
Before this commit: robot robot, 3 links, 2 joints
Links:
- added link BackLowerLeg, mass 1; collision box size=0.2 0.2 1; visual box size=0.2 0.2 1
- added link FrontLowerLeg, mass 1; collision box size=0.2 0.2 1; visual box size=0.2 0.2 1
- added link LeftLeg, mass 1; collision box size=1 0.2 0.2; visual box size=1 0.2 0.2
- added link LeftLowerLeg, mass 1; collision box size=0.2 0.2 1; visual box size=0.2 0.2 1
- added link RightLeg, mass 1; collision box size=1 0.2 0.2; visual box size=1 0.2 0.2
- added link RightLowerLeg, mass 1; collision box size=0.2 0.2 1; visual box size=0.2 0.2 1
- link BackLeg: geometry collision box size=0.2 1 0.2; visual box size=0.2 1 0.2
- link FrontLeg: geometry collision box size=0.2 1 0.2; visual box size=0.2 1 0.2
Joints:
- added joint BackLeg_BackLowerLeg: type revolute, parent BackLeg, child BackLowerLeg, origin xyz=0 -1 0 rpy=0 0 0, axis 1 0 0, limit lower=-3.14159 upper=3.14159 effort=0.0 velocity=0.0
- added joint FrontLeg_FrontLowerLeg: type revolute, parent FrontLeg, child FrontLowerLeg, origin xyz=0 1 0 rpy=0 0 0, axis 1 0 0, limit lower=-3.14159 upper=3.14159 effort=0.0 velocity=0.0
- added joint LeftLeg_LeftLowerLeg: type revolute, parent LeftLeg, child LeftLowerLeg, origin xyz=-1 0 0 rpy=0 0 0, axis 1 0 0, limit lower=-3.14159 upper=3.14159 effort=0.0 velocity=0.0
- added joint RightLeg_RightLowerLeg: type revolute, parent RightLeg, child RightLowerLeg, origin xyz=1 0 0 rpy=0 0 0, axis 1 0 0, limit lower=-3.14159 upper=3.14159 effort=0.0 velocity=0.0
- added joint Torso_LeftLeg: type revolute, parent Torso, child LeftLeg, origin xyz=-0.5 0 1 rpy=0 0 0, axis 0 1 0, limit lower=-3.14159 upper=3.14159 effort=0.0 velocity=0.0
- added joint Torso_RightLeg: type revolute, parent Torso, child RightLeg, origin xyz=0.5 0 1 rpy=0 0 0, axis 0 1 0, limit lower=-3.14159 upper=3.14159 effort=0.0 velocity=0.0
- joint Torso_BackLeg: axis 0 1 0 -> 1 0 0; origin xyz=1.0 0 1.0 rpy=0 0 0 -> xyz=0 -0.5 1.0 rpy=0 0 0
- joint Torso_FrontLeg: axis 0 1 0 -> 1 0 0; origin xyz=2 0 1 rpy=0 0 0 -> xyz=0 0.5 1 rpy=0 0 0

Commit message: commit

File: body.urdf (robot description, URDF)
Before this commit: robot robot, 9 links, 8 joints
Joints:
- joint Torso_LeftLeg: axis 0 1 0 -> 1 0 0
- joint Torso_RightLeg: axis 0 1 0 -> 1 0 0

Commit message: commit

File: body.urdf (robot description, URDF)
Before this commit: robot robot, 9 links, 8 joints
Joints:
- joint LeftLeg_LeftLowerLeg: axis 1 0 0 -> 0 1 0
- joint RightLeg_RightLowerLeg: axis 1 0 0 -> 0 1 0
- joint Torso_LeftLeg: axis 1 0 0 -> 0 1 0
- joint Torso_RightLeg: axis 1 0 0 -> 0 1 0

Commit message: commit

File: body.urdf (robot description, URDF)
Before this commit: robot robot, 9 links, 8 joints
Joints:
- joint Torso_FrontLeg: axis 1 0 0 ->  1 0 0

Commit message: commit

File: body.urdf (robot description, URDF)
Before this commit: robot robot, 9 links, 8 joints
Links:
- removed link BackLeg
- removed link BackLowerLeg
- removed link FrontLeg
- removed link FrontLowerLeg
- removed link LeftLowerLeg
- removed link RightLowerLeg
- added link Lower_LeftLeg, mass 1; collision box size=0.2 0.2 0.8; visual box size=0.2 0.2 0.8
- added link Lower_RightLeg, mass 1; collision box size=0.2 0.2 0.8; visual box size=0.2 0.2 0.8
- link LeftLeg: geometry collision box size=0.2 1 0.2; visual box size=0.2 1 0.2
- link RightLeg: geometry collision box size=0.2 1 0.2; visual box size=0.2 1 0.2
Joints:
- removed joint BackLeg_BackLowerLeg
- removed joint FrontLeg_FrontLowerLeg
- removed joint LeftLeg_LeftLowerLeg
- removed joint RightLeg_RightLowerLeg
- removed joint Torso_BackLeg
- removed joint Torso_FrontLeg
- added joint Lower_LeftLeg2: type revolute, parent LeftLeg, child Lower_LeftLeg, origin xyz=0 -0.5 -0.5 rpy=0 0 0, axis 1 0 0, limit lower=-3.14159 upper=3.14159 effort=0.0 velocity=0.0
- added joint Lower_RightLeg2: type revolute, parent RightLeg, child Lower_RightLeg, origin xyz=0 -0.5 -0.5 rpy=0 0 0, axis 1 0 0, limit lower=-3.14159 upper=3.14159 effort=0.0 velocity=0.0
- joint Torso_LeftLeg: axis 0 1 0 -> 1 0 0; origin xyz=-0.5 0 1 rpy=0 0 0 -> xyz=0 -0.8 0.5 rpy=0 0 0
- joint Torso_RightLeg: axis 0 1 0 -> 1 0 0; origin xyz=0.5 0 1 rpy=0 0 0 -> xyz=0 -0.8 0.5 rpy=0 0 0

Commit message: update

File: body.urdf (robot description, URDF)
Before this commit: robot robot, 5 links, 4 joints
Links:
- removed link LeftLeg
- removed link Lower_LeftLeg
- removed link Lower_RightLeg
- removed link RightLeg
- added link BackLeftLeg, mass 1; collision box size=0.2 1 0.2; visual box size=0.2 1 0.2
- added link BackRightLeg, mass 1; collision box size=0.2 1 0.2; visual box size=0.2 1 0.2
- added link FrontLeftLeg, mass 1; collision box size=0.2 1 0.2; visual box size=0.2 1 0.2
- added link FrontRightLeg, mass 1; collision box size=0.2 1 0.2; visual box size=0.2 1 0.2
- added link Head, mass 1; collision sphere radius=0.3; visual sphere radius=0.3
- added link LeftLeftLeg, mass 1; collision box size=1 0.2 0.2; visual box size=1 0.2 0.2
- added link LeftRightLeg, mass 1; collision box size=1 0.2 0.2; visual box size=1 0.2 0.2
- added link Lower_BackLeftLeg, mass 1; collision box size=0.2 0.2 0.8; visual box size=0.2 0.2 0.8
- added link Lower_BackRightLeg, mass 1; collision box size=0.2 0.2 0.8; visual box size=0.2 0.2 0.8
- added link Lower_FrontLeftLeg, mass 1; collision box size=0.2 0.2 0.8; visual box size=0.2 0.2 0.8
- added link Lower_FrontRightLeg, mass 1; collision box size=0.2 0.2 0.8; visual box size=0.2 0.2 0.8
- added link Lower_LeftLeftLeg, mass 1; collision box size=0.2 0.2 0.8; visual box size=0.2 0.2 0.8
- added link Lower_LeftRightLeg, mass 1; collision box size=0.2 0.2 0.8; visual box size=0.2 0.2 0.8
- added link Lower_RightLeftLeg, mass 1; collision box size=0.2 0.2 0.8; visual box size=0.2 0.2 0.8
- added link Lower_RightRightLeg, mass 1; collision box size=0.2 0.2 0.8; visual box size=0.2 0.2 0.8
- added link RightLeftLeg, mass 1; collision box size=1 0.2 0.2; visual box size=1 0.2 0.2
- added link RightRightLeg, mass 1; collision box size=1 0.2 0.2; visual box size=1 0.2 0.2
- added link Upper_Body, mass 1; collision box size=0.5 0.8 0.8; visual box size=0.5 0.8 0.8
Joints:
- removed joint Lower_LeftLeg2
- removed joint Lower_RightLeg2
- removed joint Torso_LeftLeg
- removed joint Torso_RightLeg
- added joint Head_joint: type spherical, parent Upper_Body, child Head, origin xyz=0 0 0.4 rpy=0 0 0, axis 1 0 0, limit lower=-3.14159 upper=3.14159 effort=0.0 velocity=0.0
- added joint Lower_BackLeftLeg2: type revolute, parent BackLeftLeg, child Lower_BackLeftLeg, origin xyz=0 -1 0 rpy=0 0 0, axis 1 0 0, limit lower=-3.14159 upper=3.14159 effort=0.0 velocity=0.0
- added joint Lower_BackRightLeg2: type revolute, parent BackRightLeg, child Lower_BackRightLeg, origin xyz=0 -1 0 rpy=0 0 0, axis 1 0 0, limit lower=-3.14159 upper=3.14159 effort=0.0 velocity=0.0
- added joint Lower_FrontLeftLeg2: type revolute, parent FrontLeftLeg, child Lower_FrontLeftLeg, origin xyz=0 1 0 rpy=0 0 0, axis 1 0 0, limit lower=-3.14159 upper=3.14159 effort=0.0 velocity=0.0
- added joint Lower_FrontRightLeg2: type revolute, parent FrontRightLeg, child Lower_FrontRightLeg, origin xyz=0 1 0 rpy=0 0 0, axis 1 0 0, limit lower=-3.14159 upper=3.14159 effort=0.0 velocity=0.0
- added joint Lower_LeftLeftLeg2: type revolute, parent LeftLeftLeg, child Lower_LeftLeftLeg, origin xyz=-1 0 0 rpy=0 0 0, axis 0 1 0, limit lower=-3.14159 upper=3.14159 effort=0.0 velocity=0.0
- added joint Lower_LeftRightLeg2: type revolute, parent LeftRightLeg, child Lower_LeftRightLeg, origin xyz=-1 0 0 rpy=0 0 0, axis 0 1 0, limit lower=-3.14159 upper=3.14159 effort=0.0 velocity=0.0
- added joint Lower_RightLeftLeg2: type revolute, parent RightLeftLeg, child Lower_RightLeftLeg, origin xyz=1 0 0 rpy=0 0 0, axis 0 1 0, limit lower=-3.14159 upper=3.14159 effort=0.0 velocity=0.0
- added joint Lower_RightRightLeg2: type revolute, parent RightRightLeg, child Lower_RightRightLeg, origin xyz=1 0 0 rpy=0 0 0, axis 0 1 0, limit lower=-3.14159 upper=3.14159 effort=0.0 velocity=0.0
- added joint Torso_BackLeftLeg: type revolute, parent Torso, child BackLeftLeg, origin xyz=0 -0.5 1 rpy=0 0 0, axis 1 0 0, limit lower=-3.14159 upper=3.14159 effort=0.0 velocity=0.0
- added joint Torso_BackRightLeg: type revolute, parent Torso, child BackRightLeg, origin xyz=0 -0.5 1 rpy=0 0 0, axis 1 0 0, limit lower=-3.14159 upper=3.14159 effort=0.0 velocity=0.0
- added joint Torso_FrontLeftLeg: type revolute, parent Torso, child FrontLeftLeg, origin xyz=0 0.5 1 rpy=0 0 0, axis 1 0 0, limit lower=-3.14159 upper=3.14159 effort=0.0 velocity=0.0
- added joint Torso_FrontRightLeg: type revolute, parent Torso, child FrontRightLeg, origin xyz=0 0.5 1 rpy=0 0 0, axis 1 0 0, limit lower=-3.14159 upper=3.14159 effort=0.0 velocity=0.0
- added joint Torso_LeftLeftLeg: type revolute, parent Torso, child LeftLeftLeg, origin xyz=-0.5 0 1 rpy=0 0 0, axis 0 1 0, limit lower=-3.14159 upper=3.14159 effort=0.0 velocity=0.0
- added joint Torso_LeftRightLeg: type revolute, parent Torso, child LeftRightLeg, origin xyz=-0.5 0 1 rpy=0 0 0, axis 0 1 0, limit lower=-3.14159 upper=3.14159 effort=0.0 velocity=0.0
- added joint Torso_RightLeftLeg: type revolute, parent Torso, child RightLeftLeg, origin xyz=0.5 0 1 rpy=0 0 0, axis 0 1 0, limit lower=-3.14159 upper=3.14159 effort=0.0 velocity=0.0
- added joint Torso_RightRightLeg: type revolute, parent Torso, child RightRightLeg, origin xyz=0.5 0 1 rpy=0 0 0, axis 0 1 0, limit lower=-3.14159 upper=3.14159 effort=0.0 velocity=0.0
- added joint Torso_UpperBody: type fixed, parent Torso, child Upper_Body, origin xyz=0 0 0.5 rpy=0 0 0, axis 1 0 0, limit lower=-3.14159 upper=3.14159 effort=0.0 velocity=0.0

Commit message: commit

File: body.urdf (robot description, URDF)
Before this commit: robot robot, 19 links, 18 joints
Joints:
- removed joint Lower_BackLeftLeg2
- removed joint Lower_BackRightLeg2
- removed joint Lower_FrontLeftLeg2
- removed joint Lower_FrontRightLeg2
- removed joint Lower_LeftLeftLeg2
- removed joint Lower_LeftRightLeg2
- removed joint Lower_RightLeftLeg2
- removed joint Lower_RightRightLeg2
- added joint BackLeftLeg_BackLowerLeftLeg: type revolute, parent BackLeftLeg, child Lower_BackLeftLeg, origin xyz=0 -1 0 rpy=0 0 0, axis 1 0 0, limit lower=-3.14159 upper=3.14159 effort=0.0 velocity=0.0
- added joint BackRightLeg_BackLowerRightLeg: type revolute, parent BackRightLeg, child Lower_BackRightLeg, origin xyz=0 -1 0 rpy=0 0 0, axis 1 0 0, limit lower=-3.14159 upper=3.14159 effort=0.0 velocity=0.0
- added joint FrontLeftLeg_FrontLowerLeftLeg: type revolute, parent FrontLeftLeg, child Lower_FrontLeftLeg, origin xyz=0 1 0 rpy=0 0 0, axis 1 0 0, limit lower=-3.14159 upper=3.14159 effort=0.0 velocity=0.0
- added joint FrontRightLeg_FrontLowerRightLeg: type revolute, parent FrontRightLeg, child Lower_FrontRightLeg, origin xyz=0 1 0 rpy=0 0 0, axis 1 0 0, limit lower=-3.14159 upper=3.14159 effort=0.0 velocity=0.0
- added joint LeftLeftLeg_LeftLowerLeftLeg: type revolute, parent LeftLeftLeg, child Lower_LeftLeftLeg, origin xyz=-1 0 0 rpy=0 0 0, axis 0 1 0, limit lower=-3.14159 upper=3.14159 effort=0.0 velocity=0.0
- added joint LeftRightLeg_LeftLowerRightLeg: type revolute, parent LeftRightLeg, child Lower_LeftRightLeg, origin xyz=-1 0 0 rpy=0 0 0, axis 0 1 0, limit lower=-3.14159 upper=3.14159 effort=0.0 velocity=0.0
- added joint RightLeftLeg_RightLowerLeftLeg: type revolute, parent RightLeftLeg, child Lower_RightLeftLeg, origin xyz=1 0 0 rpy=0 0 0, axis 0 1 0, limit lower=-3.14159 upper=3.14159 effort=0.0 velocity=0.0
- added joint RightRightLeg_RightLowerRightLeg: type revolute, parent RightRightLeg, child Lower_RightRightLeg, origin xyz=1 0 0 rpy=0 0 0, axis 0 1 0, limit lower=-3.14159 upper=3.14159 effort=0.0 velocity=0.0

Commit message: commit

File: body.urdf (robot description, URDF)
Before this commit: robot robot, 19 links, 18 joints
Links:
- removed link Lower_BackLeftLeg
- removed link Lower_BackRightLeg
- removed link Lower_FrontLeftLeg
- removed link Lower_FrontRightLeg
- removed link Lower_LeftLeftLeg
- removed link Lower_LeftRightLeg
- removed link Lower_RightLeftLeg
- removed link Lower_RightRightLeg
- added link BackLowerLeftLeg, mass 1; collision box size=0.2 0.2 0.8; visual box size=0.2 0.2 0.8
- added link BackLowerRightLeg, mass 1; collision box size=0.2 0.2 0.8; visual box size=0.2 0.2 0.8
- added link FrontLowerLeftLeg, mass 1; collision box size=0.2 0.2 0.8; visual box size=0.2 0.2 0.8
- added link FrontLowerRightLeg, mass 1; collision box size=0.2 0.2 0.8; visual box size=0.2 0.2 0.8
- added link LeftLowerLeftLeg, mass 1; collision box size=0.2 0.2 0.8; visual box size=0.2 0.2 0.8
- added link LeftLowerRightLeg, mass 1; collision box size=0.2 0.2 0.8; visual box size=0.2 0.2 0.8
- added link RightLowerLeftLeg, mass 1; collision box size=0.2 0.2 0.8; visual box size=0.2 0.2 0.8
- added link RightLowerRightLeg, mass 1; collision box size=0.2 0.2 0.8; visual box size=0.2 0.2 0.8
Joints:
- joint BackLeftLeg_BackLowerLeftLeg: child Lower_BackLeftLeg -> BackLowerLeftLeg
- joint BackRightLeg_BackLowerRightLeg: child Lower_BackRightLeg -> BackLowerRightLeg
- joint FrontLeftLeg_FrontLowerLeftLeg: child Lower_FrontLeftLeg -> FrontLowerLeftLeg
- joint FrontRightLeg_FrontLowerRightLeg: child Lower_FrontRightLeg -> FrontLowerRightLeg
- joint Head_joint: axis 1 0 0 -> 0 0 1 ; type spherical -> revolute
- joint LeftLeftLeg_LeftLowerLeftLeg: child Lower_LeftLeftLeg -> LeftLowerLeftLeg
- joint LeftRightLeg_LeftLowerRightLeg: child Lower_LeftRightLeg -> LeftLowerRightLeg
- joint RightLeftLeg_RightLowerLeftLeg: child Lower_RightLeftLeg -> RightLowerLeftLeg
- joint RightRightLeg_RightLowerRightLeg: child Lower_RightRightLeg -> RightLowerRightLeg

Commit message: commit

File: body.urdf (robot description, URDF)
Before this commit: robot robot, 19 links, 18 joints
Links:
- removed link BackLowerLeftLeg
- removed link BackLowerRightLeg
- removed link FrontLowerLeftLeg
- removed link FrontLowerRightLeg
- removed link LeftLowerLeftLeg
- removed link LeftLowerRightLeg
- removed link RightLowerLeftLeg
- removed link RightLowerRightLeg
- added link Lower_BackLeftLeg, mass 1; collision box size=0.2 0.2 0.8; visual box size=0.2 0.2 0.8
- added link Lower_BackRightLeg, mass 1; collision box size=0.2 0.2 0.8; visual box size=0.2 0.2 0.8
- added link Lower_FrontLeftLeg, mass 1; collision box size=0.2 0.2 0.8; visual box size=0.2 0.2 0.8
- added link Lower_FrontRightLeg, mass 1; collision box size=0.2 0.2 0.8; visual box size=0.2 0.2 0.8
- added link Lower_LeftLeftLeg, mass 1; collision box size=0.2 0.2 0.8; visual box size=0.2 0.2 0.8
- added link Lower_LeftRightLeg, mass 1; collision box size=0.2 0.2 0.8; visual box size=0.2 0.2 0.8
- added link Lower_RightLeftLeg, mass 1; collision box size=0.2 0.2 0.8; visual box size=0.2 0.2 0.8
- added link Lower_RightRightLeg, mass 1; collision box size=0.2 0.2 0.8; visual box size=0.2 0.2 0.8
Joints:
- joint BackLeftLeg_BackLowerLeftLeg: child BackLowerLeftLeg -> Lower_BackLeftLeg
- joint BackRightLeg_BackLowerRightLeg: child BackLowerRightLeg -> Lower_BackRightLeg
- joint FrontLeftLeg_FrontLowerLeftLeg: child FrontLowerLeftLeg -> Lower_FrontLeftLeg
- joint FrontRightLeg_FrontLowerRightLeg: child FrontLowerRightLeg -> Lower_FrontRightLeg
- joint Head_joint: axis 0 0 1  -> 1 0 0; type revolute -> spherical
- joint LeftLeftLeg_LeftLowerLeftLeg: child LeftLowerLeftLeg -> Lower_LeftLeftLeg
- joint LeftRightLeg_LeftLowerRightLeg: child LeftLowerRightLeg -> Lower_LeftRightLeg
- joint RightLeftLeg_RightLowerLeftLeg: child RightLowerLeftLeg -> Lower_RightLeftLeg
- joint RightRightLeg_RightLowerRightLeg: child RightLowerRightLeg -> Lower_RightRightLeg

Commit message: updated snake

File: body.urdf (robot description, URDF)
Before this commit: robot robot, 19 links, 18 joints
Links:
- removed link BackLeftLeg
- removed link BackRightLeg
- removed link FrontLeftLeg
- removed link FrontRightLeg
- removed link LeftLeftLeg
- removed link LeftRightLeg
- removed link Lower_BackLeftLeg
- removed link Lower_BackRightLeg
- removed link Lower_FrontLeftLeg
- removed link Lower_FrontRightLeg
- removed link Lower_LeftLeftLeg
- removed link Lower_LeftRightLeg
- removed link Lower_RightLeftLeg
- removed link Lower_RightRightLeg
- removed link RightLeftLeg
- removed link RightRightLeg
- removed link Torso
- removed link Upper_Body
- link Head: geometry collision sphere radius=0.02; visual sphere radius=0.02
Joints:
- removed joint BackLeftLeg_BackLowerLeftLeg
- removed joint BackRightLeg_BackLowerRightLeg
- removed joint FrontLeftLeg_FrontLowerLeftLeg
- removed joint FrontRightLeg_FrontLowerRightLeg
- removed joint Head_joint
- removed joint LeftLeftLeg_LeftLowerLeftLeg
- removed joint LeftRightLeg_LeftLowerRightLeg
- removed joint RightLeftLeg_RightLowerLeftLeg
- removed joint RightRightLeg_RightLowerRightLeg
- removed joint Torso_BackLeftLeg
- removed joint Torso_BackRightLeg
- removed joint Torso_FrontLeftLeg
- removed joint Torso_FrontRightLeg
- removed joint Torso_LeftLeftLeg
- removed joint Torso_LeftRightLeg
- removed joint Torso_RightLeftLeg
- removed joint Torso_RightRightLeg
- removed joint Torso_UpperBody

Commit message: changes to shape

File: body.urdf (robot description, URDF)
Before this commit: robot robot, 1 links, 0 joints
Links:
- removed link Head
- added link Link0, mass 1; collision box size=1 2 2; visual box size=1 2 2
- added link Link1, mass 1; collision box size=1 1 1; visual box size=1 1 1
- added link Link2, mass 1; collision box size=1 2 1; visual box size=1 2 1
- added link Link3, mass 1; collision box size=1 2 1; visual box size=1 2 1
Joints:
- added joint Link0_Link1: type revolute, parent Link0, child Link1, origin xyz=0 -1.0 0.5 rpy=0 0 0, axis 0 1 0, limit lower=-3.14159 upper=3.14159 effort=0.0 velocity=0.0
- added joint Link1_Link2: type revolute, parent Link1, child Link2, origin xyz=0 -2.0 0.5 rpy=0 0 0, axis 0 1 0, limit lower=-3.14159 upper=3.14159 effort=0.0 velocity=0.0
- added joint Link2_Link3: type revolute, parent Link2, child Link3, origin xyz=0 -2.0 0.5 rpy=0 0 0, axis 0 1 0, limit lower=-3.14159 upper=3.14159 effort=0.0 velocity=0.0

Commit message: changes to generate the snake

File: body.urdf (robot description, URDF)
Before this commit: robot robot, 4 links, 3 joints
Links:
- added link Link4, mass 1; collision box size=1 1 2; visual box size=1 1 2
- link Link0: geometry collision sphere radius=0.5; visual sphere radius=0.5
- link Link1: geometry collision sphere radius=1.0; visual sphere radius=1.0
- link Link2: geometry collision box size=1 2 2; visual box size=1 2 2
- link Link3: geometry collision box size=1 1 2; visual box size=1 1 2
Joints:
- added joint Link3_Link4: type revolute, parent Link3, child Link4, origin xyz=0 -1.0 0.5 rpy=0 0 0, axis 1 0 0, limit lower=-3.14159 upper=3.14159 effort=0.0 velocity=0.0
- joint Link0_Link1: axis 0 1 0 -> 1 0 0; origin xyz=0 -1.0 0.5 rpy=0 0 0 -> xyz=0 -0.5 0.5 rpy=0 0 0
- joint Link1_Link2: axis 0 1 0 -> 1 0 0
- joint Link2_Link3: axis 0 1 0 -> 1 0 0

Commit message: changes

File: body.urdf (robot description, URDF)
Before this commit: robot robot, 5 links, 4 joints
Links:
- added link Link5, mass 1; collision sphere radius=0.5; visual sphere radius=0.5
- added link Link6, mass 1; collision box size=2 1 2; visual box size=2 1 2
- added link Link7, mass 1; collision sphere radius=1.0; visual sphere radius=1.0
- added link Link8, mass 1; collision sphere radius=1.0; visual sphere radius=1.0
- link Link1: geometry collision box size=2 1 2; visual box size=2 1 2
- link Link3: geometry collision sphere radius=1.0; visual sphere radius=1.0
- link Link4: geometry collision sphere radius=0.5; visual sphere radius=0.5
Joints:
- added joint Link4_Link5: type revolute, parent Link4, child Link5, origin xyz=0 -1.0 0.5 rpy=0 0 0, axis 1 0 0, limit lower=-3.14159 upper=3.14159 effort=0.0 velocity=0.0
- added joint Link5_Link6: type revolute, parent Link5, child Link6, origin xyz=0 -1.0 0.5 rpy=0 0 0, axis 1 0 0, limit lower=-3.14159 upper=3.14159 effort=0.0 velocity=0.0
- added joint Link6_Link7: type revolute, parent Link6, child Link7, origin xyz=0 -1.0 0.5 rpy=0 0 0, axis 1 0 0, limit lower=-3.14159 upper=3.14159 effort=0.0 velocity=0.0
- added joint Link7_Link8: type revolute, parent Link7, child Link8, origin xyz=0 -2.0 0.5 rpy=0 0 0, axis 1 0 0, limit lower=-3.14159 upper=3.14159 effort=0.0 velocity=0.0
- joint Link1_Link2: origin xyz=0 -2.0 0.5 rpy=0 0 0 -> xyz=0 -1.0 0.5 rpy=0 0 0
- joint Link3_Link4: origin xyz=0 -1.0 0.5 rpy=0 0 0 -> xyz=0 -2.0 0.5 rpy=0 0 0

Commit message: changes

File: body.urdf (robot description, URDF)
Before this commit: robot robot, 9 links, 8 joints
Links:
- removed link Link8
- link Link0: geometry collision sphere radius=1.0; visual sphere radius=1.0
- link Link1: geometry collision sphere radius=0.5; visual sphere radius=0.5
- link Link2: geometry collision box size=2 2 2; visual box size=2 2 2
- link Link3: geometry collision box size=1 1 1; visual box size=1 1 1
- link Link4: geometry collision box size=1 1 2; visual box size=1 1 2
- link Link5: geometry collision sphere radius=1.0; visual sphere radius=1.0
- link Link6: geometry collision sphere radius=1.0; visual sphere radius=1.0
Joints:
- removed joint Link7_Link8
- joint Link0_Link1: origin xyz=0 -0.5 0.5 rpy=0 0 0 -> xyz=0 -1.0 0.5 rpy=0 0 0
- joint Link3_Link4: origin xyz=0 -2.0 0.5 rpy=0 0 0 -> xyz=0 -1.0 0.5 rpy=0 0 0
- joint Link5_Link6: origin xyz=0 -1.0 0.5 rpy=0 0 0 -> xyz=0 -2.0 0.5 rpy=0 0 0
- joint Link6_Link7: origin xyz=0 -1.0 0.5 rpy=0 0 0 -> xyz=0 -2.0 0.5 rpy=0 0 0
