Commit message: commit

File: body/body0.urdf (robot description, URDF)
Before this commit: robot robot, 5 links, 4 joints
Joints:
- joint Link0_Link1: type revolute -> prismatic
- joint Link0_Link2: axis 0 0 1 -> 0 1 0
- joint Link0_Link4: type revolute -> prismatic
- joint Link2_Link3: type revolute -> prismatic
